File: Eagle_files/Water_Schematic2_1.sch (EAGLE design)
At the start: 8 parts

Commit message: Eagle files updated
Parts:
- removed BATTERY, LIGHTSENSOR, SWITCH, TEMPERATURE: (no value), con-lstb:MA03-1
- removed MICROSD: (no value), con-lstb:MA06-1
- removed REALTIMECLOCK: (no value), con-lstb:MA04-1
- removed U$1: DIGISPARK_PRO, digistump:DIGISPARK_PRO
- added B1: ARDUINO_PRO_MINI, SparkFun-Boards:ARDUINO_PRO_MINI
- added J1: Light, SparkFun-Connectors:CONN_03
- added J2: Temp, SparkFun-Connectors:CONN_03
- added J3: Battery, SparkFun-Connectors:CONN_02POLAR
- added J6: SD, SparkFun-Connectors:CONN_06SILK_FEMALE_PTH
- added J7: RTC, SparkFun-Connectors:CONN_04POLAR
- added SW1: (no value), adafruit:SWITCH_PUSHBUTTONEVQ-PE
Connections:
- removed net DATA: LIGHTSENSOR.2, U$1.PA3
- removed net TEMP: R1.1, TEMPERATURE.2, U$1.PA7
- new net A0: B1.A0, J2.2, R1.1
- new net A3: B1.A3, J1.2
- new net BAT: J3.2, SW1.P$1
- net GND: now also B1.GND, B1.GND@2, J1.3, J2.1, J3.1, J6.6, J7.1; no longer BATTERY.3, LIGHTSENSOR.3, MICROSD.6, REALTIMECLOCK.1, SWITCH.3, TEMPERATURE.1, U$1.GND1, U$1.GND2
- net MISO: now also B1.12, J6.4; no longer MICROSD.4, U$1.PA2_MISO
- net MOSI: now also B1.*11, J6.3; no longer MICROSD.3, U$1.PA4_MOSI
- net SC: now also B1.*10, J6.1; no longer MICROSD.1, U$1.PA6_SS
- net SCK: now also B1.13, J6.2; no longer MICROSD.2, U$1.PA5_SCK
- net SCL: now also B1.A5, J7.4; no longer REALTIMECLOCK.4, U$1.PB2_SCL
- net SDA: now also B1.A4, J7.3; no longer REALTIMECLOCK.3, U$1.PB0_SDA
- net VCC: now also B1.VCC, J1.1, J2.3, J6.5, J7.2; no longer BATTERY.2, LIGHTSENSOR.1, MICROSD.5, REALTIMECLOCK.2, SWITCH.1, TEMPERATURE.3, U$1.VCC1, U$1.VCC3
- net VIN: now also B1.RAW, SW1.P$2; no longer SWITCH.2, U$1.VIN1
