File: Eagle_files/Rodney/Water_Schematic2_1.brd (EAGLE design)
At the start: 32.8 x 43.7 mm, 8 parts, among them J1 Light, J2 Temp, J3 Battery, J6 SD, J7 RTC

Commit message: Updating board
Parts:
- moved R1 6.19 mm to (22.6, 23.6)
- moved J2 6.04 mm to (26.9, 30.0), turned to 270 degrees
- moved J6 3.05 mm to (26.9, 6.10)
Routing:
- net SC: track 6.20 -> 9.25 mm
- net SCK: track 8.09 -> 11.1 mm
- net MISO: track 33.6 -> 34.3 mm
Other:
- board size 32.8 x 43.7 mm -> 33 x 43.7 mm
