File: Eagle_files/in progress/Water_Schematic2_1.sch (EAGLE design)
At the start: 12 parts

Commit message: almost there brd
Parts:
- removed ARDUINO: ARDUINO_PRO_MINI, SparkFun-Boards:ARDUINO_PRO_MINI
- added B1: ARDUINO_PRO_MINI, SparkFun-Boards_mod:ARDUINO_PRO_MINI
Connections:
- removed net A4: ARDUINO.A2, LIGHT.2
- removed net VEE: ARDUINO.RST@2, J1.3
- new net A1: B1.A1, POT2.OUT
- new net A2: B1.A2, J1.3
- new net RST: B1.RST@2
- net A0: now also B1.A0, POT1.OUT; no longer ARDUINO.A0, R1.1, TEMP.2
- net A3: now also B1.A3, LIGHT.2; no longer ARDUINO.A3, SW2.P$2
- net A6: now also B1.A6, SW2.P$2; no longer ARDUINO.A6, POT1.OUT
- net A7: now also B1.A7, R1.1, TEMP.2; no longer ARDUINO.A7, POT2.OUT
- net E: now also B1.RST; no longer ARDUINO.RST
- net GND: now also B1.GND, B1.GND@2; no longer ARDUINO.GND, ARDUINO.GND@2
- net L1: now also B1.2; no longer ARDUINO.2
- net L2: now also B1.*3; no longer ARDUINO.*3
- net L3: now also B1.4; no longer ARDUINO.4
- net L4: now also B1.*5; no longer ARDUINO.*5
- net L5: now also B1.*6; no longer ARDUINO.*6
- net L6: now also B1.7; no longer ARDUINO.7
- net L7: now also B1.8; no longer ARDUINO.8
- net L8: now also B1.*9; no longer ARDUINO.*9
- net MISO: now also B1.12; no longer ARDUINO.12
- net MOSI: now also B1.*11; no longer ARDUINO.*11
- net RS: now also B1.TXO; no longer ARDUINO.TXO
- net RW: now also B1.RXI; no longer ARDUINO.RXI
- net SC: now also B1.*10; no longer ARDUINO.*10
- net SCK: now also B1.13; no longer ARDUINO.13
- net SCL: now also B1.A5; no longer ARDUINO.A5
- net SDA: now also B1.A4; no longer ARDUINO.A4
- net VCC: now also B1.VCC; no longer ARDUINO.VCC
- net VIN: now also B1.RAW; no longer ARDUINO.RAW

Commit message: almost there!!!!!!
Connections:
- net A3: now also R1.1, TEMP.2; no longer LIGHT.2
- net A7: now also LIGHT.2; no longer R1.1, TEMP.2
Changed lines of the file:
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@@
 </segment>
 <segment>
-<wire x1="10.16" y1="63.5" x2="15.24" y2="63.5" width="0.1524" layer="91"/>
-<label x="10.16" y="63.5" size="1.778" layer="95"/>
-<pinref part="LIGHT" gate="J$1" pin="2"/>
+<wire x1="38.1" y1="33.02" x2="33.02" y2="33.02" width="0.1524" layer="91"/>
+<pinref part="R1" gate="G$1" pin="1"/>
+<label x="33.02" y="33.02" size="1.778" layer="95"/>
+<pinref part="TEMP" gate="J$1" pin="2"/>
 </segment>
 </net>
@@
 </segment>
 <segment>
-<wire x1="38.1" y1="33.02" x2="33.02" y2="33.02" width="0.1524" layer="91"/>
-<pinref part="R1" gate="G$1" pin="1"/>
-<label x="33.02" y="33.02" size="1.778" layer="95"/>
-<pinref part="TEMP" gate="J$1" pin="2"/>
+<wire x1="10.16" y1="63.5" x2="15.24" y2="63.5" width="0.1524" layer="91"/>
+<label x="10.16" y="63.5" size="1.778" layer="95"/>
+<pinref part="LIGHT" gate="J$1" pin="2"/>
 </segment>
 </net>

Commit message: got the latest schematic working
Connections:
- net A1: now also J1.3; no longer POT2.OUT
- net A2: now also POT2.OUT; no longer J1.3
- net A3: now also SW2.P$2; no longer R1.1, TEMP.2
- net A6: now also LIGHT.2; no longer SW2.P$2
- net A7: now also R1.1, TEMP.2; no longer LIGHT.2
Changed lines of the file:
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@@
 </segment>
 <segment>
-<wire x1="38.1" y1="33.02" x2="33.02" y2="33.02" width="0.1524" layer="91"/>
-<pinref part="R1" gate="G$1" pin="1"/>
-<label x="33.02" y="33.02" size="1.778" layer="95"/>
-<pinref part="TEMP" gate="J$1" pin="2"/>
+<pinref part="SW2" gate="G$1" pin="P$2"/>
+<wire x1="71.12" y1="33.02" x2="73.66" y2="33.02" width="0.1524" layer="91"/>
+<label x="71.12" y="33.02" size="1.778" layer="95"/>
 </segment>
 </net>
@@
 </segment>
 <segment>
-<pinref part="SW2" gate="G$1" pin="P$2"/>
-<wire x1="71.12" y1="33.02" x2="73.66" y2="33.02" width="0.1524" layer="91"/>
-<label x="71.12" y="33.02" size="1.778" layer="95"/>
+<wire x1="10.16" y1="63.5" x2="15.24" y2="63.5" width="0.1524" layer="91"/>
+<label x="10.16" y="63.5" size="1.778" layer="95"/>
+<pinref part="LIGHT" gate="J$1" pin="2"/>
 </segment>
 </net>
@@
 </segment>
 <segment>
-<wire x1="10.16" y1="63.5" x2="15.24" y2="63.5" width="0.1524" layer="91"/>
-<label x="10.16" y="63.5" size="1.778" layer="95"/>
-<pinref part="LIGHT" gate="J$1" pin="2"/>
+<wire x1="38.1" y1="33.02" x2="33.02" y2="33.02" width="0.1524" layer="91"/>
+<pinref part="R1" gate="G$1" pin="1"/>
+<label x="33.02" y="33.02" size="1.778" layer="95"/>
+<pinref part="TEMP" gate="J$1" pin="2"/>
 </segment>
 </net>
@@
 </segment>
 <segment>
-<pinref part="J1" gate="G$1" pin="3"/>
-<wire x1="-7.62" y1="35.56" x2="-2.54" y2="35.56" width="0.1524" layer="91"/>
-<label x="-7.62" y="35.56" size="1.778" layer="95"/>
+<pinref part="POT2" gate="G$1" pin="OUT"/>
+<wire x1="27.94" y1="76.2" x2="33.02" y2="76.2" width="0.1524" layer="91"/>
+<label x="30.48" y="76.2" size="1.778" layer="95"/>
 </segment>
 </net>
@@
 </segment>
 <segment>
-<pinref part="POT2" gate="G$1" pin="OUT"/>
-<wire x1="27.94" y1="76.2" x2="33.02" y2="76.2" width="0.1524" layer="91"/>
-<label x="30.48" y="76.2" size="1.778" layer="95"/>
+<pinref part="J1" gate="G$1" pin="3"/>
+<wire x1="-7.62" y1="35.56" x2="-2.54" y2="35.56" width="0.1524" layer="91"/>
+<label x="-7.62" y="35.56" size="1.778" layer="95"/>
 </segment>
 </net>

Commit message: attempt 2 lcd
Parts:
- removed SW2: (no value), adafruit:SWITCH_PUSHBUTTONEVQ-PE
- added R2: 220, rcl:R-US_0204/7
- added R3: 1.4k, rcl:R-US_0204/7
Connections:
- net L1 renamed D0
- net L2 renamed D1
- net L3 renamed D2
- net L4 renamed D3
- net L5 renamed D4
- net L6 renamed D5
- net L7 renamed D6
- net L8 renamed D7
- removed net A0: B1.A0, POT1.OUT
- removed net A1: B1.A1, J1.3
- removed net RST: B1.RST@2
- removed net RW: B1.RXI, J1.5
- new net BL: J1.15, R2.1
- new net V0: J1.3, R3.1
- net A3: now also POT1.OUT; no longer SW2.P$2
- net E: now also B1.RXI; no longer B1.RST
- net GND: now also J1.5, R3.2
- net VCC: now also R2.2; no longer J1.15, SW2.P$1
